File: NeuWatch.brd (EAGLE design)
At the start: 38.1 x 40.6 mm, 69 parts, among them IC1 SAMD21G18A-AUT, IC3 TPS2115, IC4 SIP32401A, IC5 MC74VHC1G14DFT, T1 846, T2 2N7002_ALT, Y1 32,768Khz

Commit message: CLR SPI
Current Limiting Resistors added to SPI
Parts:
- added R19, R25, R26: 1k, adafruit:R0402
Connections:
- new net N$15: IC1.28, R19.2
- new net N$16: IC1.26, R25.2
- new net N$17: IC1.25, R26.2
- net MISO/D12: now also R19.1; no longer IC1.28
- net MOSI/D11: now also R26.1; no longer IC1.25
- net SCK/D13: now also R25.1; no longer IC1.26
Routing:
- net N$15: track 0.00 -> 7.42 mm
- net N$16: track 0.00 -> 7.28 mm
- net N$17: track 0.00 -> 7.07 mm, vias 0 -> 2
- net SCK/D13: track 53.4 -> 47.1 mm
- net MISO/D12: track 32.9 -> 26.8 mm
- net MOSI/D11: track 52.7 -> 46.8 mm
Changed lines of the file:
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@@
 <layer number="23" name="tOrigins" color="15" fill="1" visible="yes" active="yes"/>
 <layer number="24" name="bOrigins" color="15" fill="1" visible="yes" active="yes"/>
-<layer number="25" name="tNames" color="7" fill="1" visible="no" active="yes"/>
+<layer number="25" name="tNames" color="7" fill="1" visible="yes" active="yes"/>
 <layer number="26" name="bNames" color="7" fill="1" visible="no" active="yes"/>
 <layer number="27" name="tValues" color="7" fill="1" visible="no" active="yes"/>
@@
 </element>
 <element name="C7" library="AtomTech" package="C0402" value="22pF" x="26.924" y="36.7665" smashed="yes" rot="R315">
-<attribute name="NAME" x="27.098975" y="37.811075" size="0.8128" layer="25" rot="R315"/>
+<attribute name="NAME" x="24.749475" y="38.382575" size="0.8128" layer="25" rot="R315"/>
 </element>
 <element name="C8" library="AtomTech" package="C0402" value="22pF" x="25.8445" y="35.7505" smashed="yes" rot="R315">
-<attribute name="NAME" x="24.250821875" y="35.0631875" size="0.8128" layer="25" rot="R315"/>
+<attribute name="NAME" x="23.679321875" y="37.3491875" size="0.8128" layer="25" rot="R315"/>
 </element>
 <element name="C6" library="AtomTech" package="C0402" value="100nF" x="10.414" y="23.749" smashed="yes" rot="R90">
@@
 </element>
 <element name="SWD" library="Neutrino-" package="ARDUINO-NEUTRINO-082_CONNETTORI_PINHEAD-2X5-P127" value="PINHEAD-2x5-P1.27" x="30.607" y="38.5445" smashed="yes" rot="R270">
-<attribute name="NAME" x="29.591" y="36.195" size="0.8128" layer="25" font="vector" ratio="16"/>
+<attribute name="NAME" x="34.0995" y="38.9255" size="0.8128" layer="25" font="vector" ratio="16"/>
 <attribute name="VALUE" value="PINHEAD-2x5-P1.27" x="26.162" y="41.7195" size="0.635" layer="27" font="vector" ratio="16" rot="R270"/>
 </element>
@@
 <element name="R18" library="rcl" package="R0402" value="4.7k" x="18.3515" y="12.319" rot="R270"/>
 <element name="C21" library="AtomTech" package="C0402" value="470nf" x="18.415" y="5.842" rot="R270"/>
+<element name="R19" library="adafruit" package="R0402" value="1k" x="28.194" y="19.685" smashed="yes" rot="R90">
+<attribute name="NAME" x="28.6385" y="16.256" size="0.8128" layer="25" rot="R90"/>
+<attribute name="VALUE" x="30.226" y="19.05" size="1.27" layer="27" rot="R90"/>
+</element>
+<element name="R25" library="adafruit" package="R0402" value="1k" x="26.9875" y="19.685" smashed="yes" rot="R90">
+<attribute name="NAME" x="27.432" y="16.256" size="0.8128" layer="25" rot="R90"/>
+<attribute name="VALUE" x="29.0195" y="19.05" size="1.27" layer="27" rot="R90"/>
+</element>
+<element name="R26" library="adafruit" package="R0402" value="1k" x="25.781" y="19.685" smashed="yes" rot="R90">
+<attribute name="NAME" x="26.0985" y="16.256" size="0.8128" layer="25" rot="R90"/>
+<attribute name="VALUE" x="27.813" y="19.05" size="1.27" layer="27" rot="R90"/>
+</element>
 </elements>
 <signals>
@@
 </signal>
 <signal name="SCK/D13">
-<contactref element="IC1" pad="26"/>
 <contactref element="OLED" pad="P$8"/>
 <contactref element="OLED" pad="P$3"/>
@@
 <wire x1="27.8765" y1="1.7145" x2="27.8765" y2="2.2225" width="0.4064" layer="16"/>
 <wire x1="27.8765" y1="2.2225" x2="27.813" y2="2.286" width="0.4064" layer="16"/>
-<wire x1="31.340390625" y1="23.135628125" x2="31.8135" y2="22.66251875" width="0.254" layer="1"/>
-<wire x1="31.8135" y1="22.66251875" x2="31.8135" y2="21.336" width="0.254" layer="1"/>
-<wire x1="31.8135" y1="21.336" x2="25.7175" y2="15.24" width="0.254" layer="1"/>
 <wire x1="25.7175" y1="15.24" x2="22.606" y2="15.24" width="0.254" layer="1"/>
 <via x="22.606" y="15.24" extent="1-16" drill="0.3302"/>
@@
 <wire x1="12.192" y1="4.0005" x2="12.573" y2="3.6195" width="0.254" layer="2"/>
 <wire x1="12.573" y1="3.6195" x2="12.573" y2="2.286" width="0.254" layer="2"/>
+<contactref element="R25" pad="1"/>
+<wire x1="26.9875" y1="19.035" x2="26.9875" y2="16.51" width="0.254" layer="1"/>
+<wire x1="26.9875" y1="16.51" x2="25.7175" y2="15.24" width="0.254" layer="1"/>
 </signal>
 <signal name="3.3V">
@@
 </signal>
 <signal name="MISO/D12">
-<contactref element="IC1" pad="28"/>
 <contactref element="OLED" pad="P$4"/>
-<wire x1="32.047496875" y1="23.842734375" x2="32.512" y2="23.37823125" width="0.254" layer="1"/>
-<wire x1="32.512" y1="23.37823125" x2="32.512" y2="21.1455" width="0.254" layer="1"/>
-<wire x1="32.512" y1="21.1455" x2="29.083" y2="17.7165" width="0.254" layer="1"/>
 <wire x1="29.083" y1="17.7165" x2="29.083" y2="15.5575" width="0.254" layer="1"/>
 <via x="29.083" y="15.5575" extent="1-16" drill="0.3302"/>
@@
 <wire x1="25.781" y1="10.922" x2="27.6225" y2="10.922" width="0.254" layer="15"/>
 <wire x1="27.6225" y1="10.922" x2="29.083" y2="12.3825" width="0.254" layer="15"/>
+<contactref element="R19" pad="1"/>
+<wire x1="28.194" y1="19.035" x2="28.194" y2="18.6055" width="0.254" layer="1"/>
+<wire x1="28.194" y1="18.6055" x2="29.083" y2="17.7165" width="0.254" layer="1"/>
 </signal>
 <signal name="MOSI/D11">
-<contactref element="IC1" pad="25"/>
 <contactref element="OLED" pad="P$9"/>
 <contactref element="OLED" pad="P$2"/>
@@
 <wire x1="9.9695" y1="1.778" x2="9.9695" y2="2.2225" width="0.4064" layer="1"/>
 <wire x1="9.9695" y1="2.2225" x2="10.033" y2="2.286" width="0.4064" layer="1"/>
-<wire x1="30.9868375" y1="22.782071875" x2="24.524265625" y2="16.3195" width="0.254" layer="1"/>
 <wire x1="24.524265625" y1="16.3195" x2="21.971" y2="16.3195" width="0.254" layer="1"/>
 <wire x1="21.971" y1="16.3195" x2="21.3995" y2="15.748" width="0.254" layer="1"/>
@@
 <wire x1="17.7165" y1="2.4765" x2="17.8435" y2="2.3495" width="0.254" layer="1"/>
 <wire x1="17.8435" y1="2.3495" x2="17.8435" y2="0.9525" width="0.254" layer="1"/>
+<contactref element="R26" pad="1"/>
+<wire x1="25.781" y1="19.035" x2="25.781" y2="17.576234375" width="0.254" layer="1"/>
+<wire x1="25.781" y1="17.576234375" x2="24.524265625" y2="16.3195" width="0.254" layer="1"/>
 </signal>
 <signal name="SS/D10">
@@
 <wire x1="20.447" y1="36.576" x2="20.447" y2="38.227" width="0.6096" layer="16"/>
 </signal>
+<signal name="N$15">
+<contactref element="IC1" pad="28"/>
+<contactref element="R19" pad="2"/>
+<wire x1="32.047496875" y1="23.842734375" x2="32.047496875" y2="23.832503125" width="0.254" layer="1"/>
+<wire x1="32.047496875" y1="23.832503125" x2="32.512" y2="23.368" width="0.254" layer="1"/>
+<wire x1="32.512" y1="23.368" x2="32.512" y2="21.463" width="0.254" layer="1"/>
+<wire x1="32.512" y1="21.463" x2="31.3055" y2="20.2565" width="0.254" layer="1"/>
+<wire x1="31.3055" y1="20.2565" x2="28.2725" y2="20.2565" width="0.254" layer="1"/>
+<wire x1="28.2725" y1="20.2565" x2="28.194" y2="20.335" width="0.254" layer="1"/>
+</signal>
+<signal name="N$16">
+<contactref element="IC1" pad="26"/>
+<contactref element="R25" pad="2"/>
+<wire x1="31.340390625" y1="23.135628125" x2="31.347371875" y2="23.135628125" width="0.254" layer="1"/>
+<wire x1="31.347371875" y1="23.135628125" x2="31.877" y2="22.606" width="0.254" layer="1"/>
+<wire x1="31.877" y1="22.606" x2="31.877" y2="21.717" width="0.254" layer="1"/>
+<wire x1="31.877" y1="21.717" x2="31.4325" y2="21.2725" width="0.254" layer="1"/>
+<wire x1="31.4325" y1="21.2725" x2="27.6225" y2="21.2725" width="0.254" layer="1"/>
+<wire x1="27.6225" y1="21.2725" x2="27.051" y2="20.701" width="0.254" layer="1"/>
+<wire x1="27.051" y1="20.701" x2="27.051" y2="20.3985" width="0.254" layer="1"/>
+<wire x1="27.051" y1="20.3985" x2="26.9875" y2="20.335" width="0.254" layer="1"/>
+</signal>
+<signal name="N$17">
+<contactref element="IC1" pad="25"/>
+<contactref element="R26" pad="2"/>
+<wire x1="30.9868375" y1="22.782071875" x2="30.846571875" y2="22.782071875" width="0.254" layer="1"/>
+<wire x1="30.846571875" y1="22.782071875" x2="30.353" y2="22.2885" width="0.254" layer="1"/>
+<via x="30.353" y="22.2885" extent="1-16" drill="0.3302" diameter="0.508"/>
+<wire x1="30.353" y1="22.2885" x2="30.353" y2="21.0185" width="0.254" layer="15"/>
+<wire x1="30.353" y1="21.0185" x2="29.845" y2="20.5105" width="0.254" layer="15"/>
+<wire x1="29.845" y1="20.5105" x2="25.781" y2="20.5105" width="0.254" layer="15"/>
+<via x="25.781" y="20.5105" extent="1-16" drill="0.3302" diameter="0.508"/>
+<wire x1="25.781" y1="20.5105" x2="25.781" y2="20.335" width="0.254" layer="1"/>
+</signal>
 </signals>
